File: monitor/monitor.kicad_sch (KiCad schematic)
At the start: 0 parts

Commit message: monitor functionality v1.0
Parts:
- added A1: Arduino_Uno_R4_WiFi_Shield, PCM_arduino-library:Arduino_Uno_R4_WiFi_Shield, symbol arduino-library:Arduino_Uno_R4_WiFi_Shield
- added DS1: LCD16X2_I2C, WC1602A, symbol lcd16x2_i2c:LCD16X2_I2C
- added SW1, SW2, SW3, SW4: SW_Push, symbol Switch:SW_Push
- added U1: SensorSoilMoisture, symbol ekayudhi:SensorSoilMoisture
Connections:
- new net: A1.D5, SW2.1
- new net: A1.D7, SW4.1
- new net: A1.D4, SW1.1
- new net: A1.A4, DS1.3 (SDA)
- new net: A1.A5, DS1.4 (SCL)
- new net: A1.D2, U1.2 (VCC)
- new net: A1.A0, U1.3 (OUT)
- new net: A1.D6, SW3.1
- new net +5V: A1.5V1 (5V), DS1.1 (VSS)
- new net GND: A1.GND1 (GND), DS1.2 (VDD), SW1.2, SW2.2, SW3.2, SW4.2, U1.1 (GND)
