File: hardware/kicad/plant_watering.kicad_pcb (KiCad board)
At the start: 2 copper layers, 118 x 112 mm, 49 parts, among them J1 USB-C POWER IN (5V charger), J10 Pump2_12V, J11 Pump3_12V, J12 Pump4_12V, J13 Pump5_12V, J14 Pump6_12V, J15 Float switch (water level), J2 UI MODULE, J3 Sensor1 (GND,VCC,DIS,OUT), J4 Sensor2 (GND,VCC,DIS,OUT), J5 Sensor3 (GND,VCC,DIS,OUT), J6 Sensor4 (GND,VCC,DIS,OUT), J7 Sensor5 (GND,VCC,DIS,OUT), J8 Sensor6 (GND,VCC,DIS,OUT), J9 Pump1_12V, Q1 IRLZ44N, Q2 IRLZ44N, Q3 IRLZ44N, Q4 IRLZ44N, Q5 IRLZ44N, Q6 IRLZ44N, U1 YD-ESP32-23

Commit message: Mount UI module on the PCB, panel USB-C input, extra mounting holes
- J2: replace the JST-XH 9-pin with a 1x9 2.54 mm socket plus the UI
  module's four M3 standoff holes (new UI_module_OLED_EC11 footprint);
  the module plugs in face-up left of the ESP32 and screws down
- Board widened to 143 x 112 mm for the module; UI nets rerouted,
  corner holes moved, three extra M3 holes beside J3-J8 against flex
- J1: JST-PH 6-pin for a panel-mount USB-C socket cable
- MT3608 footprint updated to measured hole spacing (26 x 13 mm)
- README/BOM: UI module photo and mounting notes, ESP pinout and
  IN-OUT jumper warning, 1:1 printable board PDF

Co-Authored-By: Claude Opus 5.5 <noreply@anthropic.com>
Parts:
- added MH5: MountingHole_3.2mm_M3, MountingHole:MountingHole_3.2mm_M3, F.Cu at (108.0, 51.0)
- added MH6: MountingHole_3.2mm_M3, MountingHole:MountingHole_3.2mm_M3, F.Cu at (108.0, 85.0)
- added MH7: MountingHole_3.2mm_M3, MountingHole:MountingHole_3.2mm_M3, F.Cu at (108.0, 119.0)
- J1: value USB-C POWER IN (5V charger) -> USB-C panel cable (PH2.0 6P); footprint Connector_USB:USB_C_Receptacle_GCT_USB4125-xx-x-0190_6P_TopMnt_Horizontal -> Connector_JST:JST_PH_B6B-PH-K_1x06_P2.00mm_Vertical
- J2: footprint Connector_JST:JST_XH_B9B-XH-A_1x09_P2.50mm_Vertical -> plant_watering_parts:UI_module_OLED_EC11
- MH1, MH2, MH3, MH4: value MountingHole_3.2mm -> MountingHole_3.2mm_M3; footprint MountingHole:MountingHole_3.2mm -> MountingHole:MountingHole_3.2mm_M3
- moved MH1 25.0 mm to (20.0, 35.0)
- moved MH3 25.0 mm to (20.0, 137.0)
- moved J1 5.83 mm to (47.5, 45.0)
- moved J2 3.90 mm to (51.0, 77.5)
Routing:
- net +3V3: track 173.3 -> 158.3 mm
- net Net-(J2-Pad1): track 71.1 -> 79.2 mm
- net Net-(J2-Pad6): track 25.3 -> 17.2 mm
- net Net-(J2-Pad5): track 19.5 -> 11.6 mm
- net Net-(J2-Pad3): track 52.1 -> 44.7 mm
- net Net-(J2-Pad4): track 14.4 -> 20.3 mm
- net +5V: track 132.4 -> 128.6 mm
- net CC2: track 12.9 -> 9.57 mm
- net Net-(J2-Pad2): track 47.5 -> 50.5 mm
- net CC1: track 11.3 -> 8.74 mm
- net Net-(J2-Pad7): track 42.0 -> 40.0 mm
Other:
- board size 118 x 112 mm -> 143 x 112 mm
